File: nand1/nand1.sch (KiCad schematic (older format))
At the start: 14 parts, among them J1 JACK-DC, J2 JACK-MONO, U1 4093

Commit message: Made pcblayout for etching
Parts:
- added LDR1: LDR, Z-FP:Jack_Instrument, symbol 4ms-passives:LDR
- C1, C2: value CP1_Small -> 1uF
- C3: value CP1_Small -> 470nF
- C4: value CP1_Small -> 10uF
- J1: footprint zfoot:Jack_DC -> Z-FP:Jack_DC; symbol zMECH:JACK-DC -> nand1-rescue:JACK-DC-zMECH
- J2: footprint zfoot:Jack_Instrument_Bigger -> Z-FP:Jack_Instrument; symbol zMECH:JACK-TIP_GND -> nand1-rescue:JACK-TIP_GND-zMECH
- R1: value R -> 15K
- R2, R3: value R -> 1.5K
- RV1, RV2, RV3: value POT -> TrimPot_T73YEt_10k; footprint zfoot:Pot_Wired -> 4ms_Potentiometer:Pot_Trim_7x6.6mm_T73YE; symbol 4ms-mech:POT -> 4ms_Potentiometer:TrimPot_T73YEt_10k; Display (none) -> 10k; Manufacturer (none) -> Vishay; Part Number (none) -> T73YE103KT20; Specifications (none) -> Trimpot, TH, 10k, single turn, square
Connections:
- net +9V: now also LDR1.1; no longer J1.1 (V)
- new net: J1.1 (V), LDR1.2
Other:
- moved on the sheet: J1
